File: board/Synchronizer.kicad_sch (KiCad schematic)
At the start: 52 parts, among them J1 POWER, J2 Conn_01x14, J3 SENSE COIL, J4 Barrel_Jack_Switch, J5 DRIVE COIL, Q1 2N3904, Q2 2N3906, Q3 IRF9540N, Q4 2N3904, U1 Pico, U2 LM7805_TO220, U3 LM358

Commit message: Add R22/C10 snubber across the drive FET drain
R22 (10R) and C10 (100 nF) in series from the Q3 drain node to ground,
damping the ringing when the P-channel FET switches the drive coil off.
They sit on the junction between Q3's drain and R6, so the snubber sees the
switching node itself rather than the coil terminal, which already has D2
across it.

Schematic gains R22, C10, #PWR026 and the wiring to reach them; the PCB
gains their footprints and the new Net-(C10-Pad2).

D2, J5 and R18 shifted a few millimetres to open up room in the drive-coil
corner, and U2 moved slightly. No other footprint changed position, nothing
was removed, and the board is still single-sided with no vias.

Regenerated from the edited design: gerbers, drill files, the schematic PDF,
the board render, and the footprint info cache. Most of the diff in the
.kicad_pcb is the refilled copper zones rather than anything logical.

Co-Authored-By: Claude Opus 5 <noreply@anthropic.com>
Claude-Session: https://claude.ai/code/session_01AQX6646joaK2TkbMXHZigW
Parts:
- added C10: 100 nF, Capacitor_THT:C_Rect_L7.0mm_W2.5mm_P5.00mm, symbol Device:C_Small
- added R22: 10R, Resistor_THT:R_Axial_DIN0207_L6.3mm_D2.5mm_P7.62mm_Horizontal, symbol Device:R
Connections:
- net GND: now also R22.2
- net at Q3.2 (D), R6.2: now also C10.1
- new net: C10.2, R22.1
Changed lines of the file:
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@@
   (junction (at 254 60.96) (diameter 0) (color 0 0 0 0)
   )
+  (junction (at 207.01 121.285) (diameter 0) (color 0 0 0 0)
+  )
   (junction (at 126.365 124.46) (diameter 0) (color 0 0 0 0)
   )
@@
     (stroke (width 0) (type default))
   )
+  (wire (pts (xy 171.45 123.825) (xy 171.45 121.285))
+    (stroke (width 0) (type default))
+  )
   (wire (pts (xy 44.45 47.625) (xy 48.26 47.625))
     (stroke (width 0) (type default))
@@
     (stroke (width 0) (type default))
   )
+  (wire (pts (xy 171.45 138.43) (xy 171.45 140.335))
+    (stroke (width 0) (type default))
+  )
   (wire (pts (xy 90.805 167.64) (xy 95.885 167.64))
     (stroke (width 0) (type default))
@@
     (stroke (width 0) (type default))
   )
+  (wire (pts (xy 171.45 128.905) (xy 171.45 130.81))
+    (stroke (width 0) (type default))
+  )
   (wire (pts (xy 98.425 142.24) (xy 98.425 149.86))
     (stroke (width 0) (type default))
@@
   )
   (wire (pts (xy 95.885 129.54) (xy 90.805 129.54))
+    (stroke (width 0) (type default))
+  )
+  (wire (pts (xy 171.45 121.285) (xy 207.01 121.285))
     (stroke (width 0) (type default))
   )
@@
         (path "/0301afe8-2926-4121-93b1-45e55e088589"
           (reference "J4") (unit 1)
+        )
+      )
+    )
+  )
+  (symbol (lib_id "power:GND") (at 171.45 140.335 0) (unit 1)
+    (in_bom yes) (on_board yes) (dnp no) (fields_autoplaced)
+    (property "Reference" "#PWR026" (at 171.45 146.685 0)
+      (effects (font (size 1.27 1.27)) hide)
+    )
+    (property "Value" "GND" (at 171.45 145.415 0)
+      (effects (font (size 1.27 1.27)))
+    )
+    (property "Footprint" "" (at 171.45 140.335 0)
+      (effects (font (size 1.27 1.27)) hide)
+    )
+    (property "Datasheet" "" (at 171.45 140.335 0)
+      (effects (font (size 1.27 1.27)) hide)
+    )
+    (pin "1")
+    (instances
+      (project "Synchronizer"
+        (path "/0301afe8-2926-4121-93b1-45e55e088589"
+          (reference "#PWR026") (unit 1)
         )
       )
@@
     )
   )
+  (symbol (lib_id "Device:C_Small") (at 171.45 126.365 0) (unit 1)
+    (in_bom yes) (on_board yes) (dnp no) (fields_autoplaced)
+    (property "Reference" "C10" (at 173.99 125.1013 0)
+      (effects (font (size 1.27 1.27)) (justify left))
+    )
+    (property "Value" "100 nF" (at 173.99 127.6413 0)
+      (effects (font (size 1.27 1.27)) (justify left))
+    )
+    (property "Footprint" "Capacitor_THT:C_Rect_L7.0mm_W2.5mm_P5.00mm" (at 171.45 126.365 0)
+      (effects (font (size 1.27 1.27)) hide)
+    )
+    (property "Datasheet" "~" (at 171.45 126.365 0)
+      (effects (font (size 1.27 1.27)) hide)
+    )
+    (pin "2")
+    (pin "1")
+    (instances
+      (project "Synchronizer"
+        (path "/0301afe8-2926-4121-93b1-45e55e088589"
+          (reference "C10") (unit 1)
+        )
+      )
+    )
+  )
   (symbol (lib_id "power:+12V") (at 48.26 47.625 0) (unit 1)
     (in_bom yes) (on_board yes) (dnp no) (fields_autoplaced)
@@
         )
       )
+    )
+  )
+  (symbol (lib_id "Device:R") (at 171.45 134.62 0) (unit 1)
+    (in_bom yes) (on_board yes) (dnp no)
+    (property "Reference" "R22" (at 173.99 137.16 90)
+      (effects (font (size 1.27 1.27)) (justify left))
+    )
+    (property "Value" "10R" (at 171.45 136.525 90)
+      (effects (font (size 1.27 1.27)) (justify left))
+    )
+    (property "Footprint" "Resistor_THT:R_Axial_DIN0207_L6.3mm_D2.5mm_P7.62mm_Horizontal" (at 169.672 134.62 90)
+      (effects (font (size 1.27 1.27)) hide)
+    )
+    (property "Datasheet" "~" (at 171.45 134.62 0)
+      (effects (font (size 1.27 1.27)) hide)
+    )
+    (pin "2")
+    (pin "1")
+    (instances
+      (project "Synchronizer"
+        (path "/0301afe8-2926-4121-93b1-45e55e088589"
+          (reference "R22") (unit 1)
+        )
+      )

Commit message: board/CAD: schematic and PCB revisions, add coil bobbin model
board/: schematic and PCB updates (new connector and polarized cap, power
rail reworked in places), regenerated gerbers/drill files, updated
schematic PDF and board render.

CAD/: revise WeightedElectromagnetHolder, add CoilBobbin (model + STL).

Co-Authored-By: Claude Sonnet 5 <noreply@anthropic.com>
Claude-Session: https://claude.ai/code/session_01AQX6646joaK2TkbMXHZigW
Parts:
- added C12: 1000 uF, Capacitor_THT:CP_Radial_D8.0mm_P2.50mm, symbol Device:C_Polarized_Small
- added J6: Conn_01x03, Connector_PinHeader_2.54mm:PinHeader_1x03_P2.54mm_Vertical, symbol Connector_Generic:Conn_01x03
- C6: value 100 pF -> 30 pF
- D3, D4: value 1N4148 -> 1N5819; footprint Diode_THT:D_DO-35_SOD27_P7.62mm_Horizontal -> Diode_THT:D_DO-41_SOD81_P7.62mm_Horizontal
- R10, R8: value 100k -> 10k
- R14: value 100k -> 33k
- R19: value 10k -> 330R
- R5: value 10k -> 100k
- R9: value 10k -> 1k
Connections:
- net +12V: now also C12.1; no longer Q2.1 (E), R8.1
- net +5V: now also Q2.1 (E), R8.1
- net GND: now also C12.2, J6.3 (Pin_3)
- net OPSUPPLY: now also J6.2 (Pin_2)
- net +3V3: now reaches D7.1 (K), D8.1 (K), R1.1, U1.36 (3V3)
- net +3V3: now also J6.1 (Pin_1)
